Commit message: feat: add spidy robot URDF description, MuJoCo model, and generation scripts

File: URDF/spidy_description/urdf/spidy.urdf (robot description, URDF)
Before this commit: robot spidy, 17 links, 16 joints
Joints:
- removed joint bl_hip_pitch
- removed joint bl_hip_yaw
- removed joint br_hip_pitch
- removed joint br_hip_yaw
- removed joint fl_hip_pitch
- removed joint fl_hip_yaw
- removed joint fr_hip_pitch
- removed joint fr_hip_yaw
- added joint bl_claw: type revolute, parent bl_femur, child bl_tibia, origin xyz=0 0.0558 0 rpy=0 0 0, axis 1 0 0, limit lower=-1.5707963267948966 upper=1.5707963267948966 effort=0.21 velocity=13.0
- added joint bl_hip: type revolute, parent base_link, child bl_coxa, origin xyz=-0.06 0.05 0 rpy=0 0 0, axis 0 0 1, limit lower=-1.5707963267948966 upper=1.5707963267948966 effort=0.21 velocity=13.0
- added joint br_claw: type revolute, parent br_femur, child br_tibia, origin xyz=0 -0.0558 0 rpy=0 0 0, axis 1 0 0, limit lower=-1.5707963267948966 upper=1.5707963267948966 effort=0.21 velocity=13.0
- added joint br_hip: type revolute, parent base_link, child br_coxa, origin xyz=-0.06 -0.05 0 rpy=0 0 0, axis 0 0 1, limit lower=-1.5707963267948966 upper=1.5707963267948966 effort=0.21 velocity=13.0
- added joint fl_claw: type revolute, parent fl_femur, child fl_tibia, origin xyz=0 0.0558 0 rpy=0 0 0, axis 1 0 0, limit lower=-1.5707963267948966 upper=1.5707963267948966 effort=0.21 velocity=13.0
- added joint fl_hip: type revolute, parent base_link, child fl_coxa, origin xyz=0.06 0.05 0 rpy=0 0 0, axis 0 0 1, limit lower=-1.5707963267948966 upper=1.5707963267948966 effort=0.21 velocity=13.0
- added joint fr_claw: type revolute, parent fr_femur, child fr_tibia, origin xyz=0 -0.0558 0 rpy=0 0 0, axis 1 0 0, limit lower=-1.5707963267948966 upper=1.5707963267948966 effort=0.21 velocity=13.0
- added joint fr_hip: type revolute, parent base_link, child fr_coxa, origin xyz=0.06 -0.05 0 rpy=0 0 0, axis 0 0 1, limit lower=-1.5707963267948966 upper=1.5707963267948966 effort=0.21 velocity=13.0
- joint bl_knee: child bl_tibia -> bl_femur; origin xyz=0 0.0558 0 rpy=0 0 0 -> xyz=0 0.0342 0 rpy=0 0 0; parent bl_femur -> bl_coxa
- joint br_knee: child br_tibia -> br_femur; origin xyz=0 -0.0558 0 rpy=0 0 0 -> xyz=0 -0.0342 0 rpy=0 0 0; parent br_femur -> br_coxa
- joint fl_knee: child fl_tibia -> fl_femur; origin xyz=0 0.0558 0 rpy=0 0 0 -> xyz=0 0.0342 0 rpy=0 0 0; parent fl_femur -> fl_coxa
- joint fr_knee: child fr_tibia -> fr_femur; origin xyz=0 -0.0558 0 rpy=0 0 0 -> xyz=0 -0.0342 0 rpy=0 0 0; parent fr_femur -> fr_coxa

File: URDF/spidy_description/urdf/spidy.urdf.xacro (robot description, xacro)
@@ -6,8 +6,10 @@
   tibias pointing straight down.
   Kinematic tree, per leg (L = fl / fr / bl / br):
-    base_link -[L_hip_yaw  z]-> L_coxa -[L_hip_pitch x]-> L_femur
-              -[L_knee     x]-> L_tibia -[fixed]-> L_foot
-  Axis convention: every leg uses the SAME axes (yaw +z, pitch +x, knee +x).
-  So +hip_pitch lifts a LEFT leg but lowers a RIGHT leg. The mirroring is
+    base_link -[L_hip  z]-> L_coxa -[L_knee x]-> L_femur
+              -[L_claw x]-> L_tibia -[fixed]-> L_foot
+  Joint names: hip = swings the leg forward/back (yaw), knee = lifts it
+  (pitch), claw = bends the tibia. Firmware calls them HIP / KNEE / ANKLE.
+  Axis convention: every leg uses the SAME axes (hip +z, knee +x, claw +x).
+  So +knee lifts a LEFT leg but lowers a RIGHT leg. The mirroring is
   handled in the IK/gait code, not hidden in the URDF (same convention as
   Unitree/ANYmal descriptions).
@@ -60,6 +62,6 @@
        sy     : +1 left,  -1 right                                           -->
   <xacro:macro name="leg" params="prefix sx sy">
-    <!-- hip yaw: servo m1 is screwed to the chassis, its horn turns the coxa -->
-    <joint name="${prefix}_hip_yaw" type="revolute">
+    <!-- hip (yaw): servo m1 is screwed to the chassis, its horn turns the coxa -->
+    <joint name="${prefix}_hip" type="revolute">
       <parent link="base_link"/>
       <child  link="${prefix}_coxa"/>
@@ -80,6 +82,6 @@
       </inertial>
     </link>
-    <!-- hip pitch: servo m2 sits in the coxa bracket, its horn drives the femur link -->
-    <joint name="${prefix}_hip_pitch" type="revolute">
+    <!-- knee (pitch): servo m2 sits in the coxa bracket, its horn drives the femur link -->
+    <joint name="${prefix}_knee" type="revolute">
       <parent link="${prefix}_coxa"/>
       <child  link="${prefix}_femur"/>
@@ -100,7 +102,7 @@
       </inertial>
     </link>
-    <!-- knee: servo m3 is screwed into the claw; its horn is fixed to the femur
+    <!-- claw: servo m3 is screwed into the claw; its horn is fixed to the femur
          link, so the servo BODY rotates with the tibia. Same joint either way. -->
-    <joint name="${prefix}_knee" type="revolute">
+    <joint name="${prefix}_claw" type="revolute">
       <parent link="${prefix}_femur"/>
       <child  link="${prefix}_tibia"/>

Commit message: feat: add spidy robot model configuration and simulation files

File: URDF/spidy_description/urdf/spidy.urdf (robot description, URDF)
Before this commit: robot spidy, 17 links, 16 joints
Links:
- link base_link: mass 0.524658 -> 0.517075
- link bl_coxa: mass 0.021068 -> 0.0200143
- link bl_femur: mass 0.0112014 -> 0.00891947
- link bl_tibia: mass 0.0185889 -> 0.0179021
- link br_coxa: mass 0.021068 -> 0.0200143
- link br_femur: mass 0.0112014 -> 0.00891947
- link br_tibia: mass 0.0185889 -> 0.0179021
- link fl_coxa: mass 0.021068 -> 0.0200143
- link fl_femur: mass 0.0112014 -> 0.00891947
- link fl_tibia: mass 0.0185889 -> 0.0179021
- link fr_coxa: mass 0.021068 -> 0.0200143
- link fr_femur: mass 0.0112014 -> 0.00891947
- link fr_tibia: mass 0.0185889 -> 0.0179021

File: URDF/spidy_description/urdf/spidy_generated.xacro (robot description, xacro)
@@ -13,43 +13,43 @@
   <xacro:property name="stack_box_xyz"  value="0.00411249 0 0.0347"/>
   <xacro:property name="stack_box_size" value="0.1428 0.086 0.075"/>
-  <xacro:property name="base_mass" value="0.524658"/>
-  <xacro:property name="base_cx" value="0.0118298"/>
-  <xacro:property name="base_cy" value="-0.000136744"/>
-  <xacro:property name="base_cz" value="0.020099"/>
-  <xacro:property name="base_ixx" value="8.5234e-04"/>
-  <xacro:property name="base_iyy" value="1.3390e-03"/>
-  <xacro:property name="base_izz" value="1.1356e-03"/>
-  <xacro:property name="base_ixy" value="3.8002e-06"/>
-  <xacro:property name="base_ixz" value="-5.4712e-05"/>
-  <xacro:property name="base_iyz" value="-1.3324e-06"/>
-  <xacro:property name="coxa_mass" value="0.021068"/>
-  <xacro:property name="coxa_cx" value="-0.00141624"/>
-  <xacro:property name="coxa_cy" value="0.0287927"/>
-  <xacro:property name="coxa_cz" value="-0.00446"/>
-  <xacro:property name="coxa_ixx" value="4.6563e-06"/>
-  <xacro:property name="coxa_iyy" value="3.4341e-06"/>
-  <xacro:property name="coxa_izz" value="3.7524e-06"/>
-  <xacro:property name="coxa_ixy" value="2.1063e-07"/>
-  <xacro:property name="coxa_ixz" value="8.4111e-09"/>
-  <xacro:property name="coxa_iyz" value="1.8597e-07"/>
-  <xacro:property name="femur_mass" value="0.0112014"/>
-  <xacro:property name="femur_cx" value="-0.00536283"/>
-  <xacro:property name="femur_cy" value="0.0278179"/>
-  <xacro:property name="femur_cz" value="6.30165e-10"/>
-  <xacro:property name="femur_ixx" value="3.3434e-06"/>
-  <xacro:property name="femur_iyy" value="3.6520e-06"/>
-  <xacro:property name="femur_izz" value="6.6136e-06"/>
-  <xacro:property name="femur_ixy" value="1.4699e-08"/>
-  <xacro:property name="femur_ixz" value="5.8266e-14"/>
+  <xacro:property name="base_mass" value="0.517075"/>
+  <xacro:property name="base_cx" value="0.0121647"/>
+  <xacro:property name="base_cy" value="-0.000138725"/>
+  <xacro:property name="base_cz" value="0.0231342"/>
+  <xacro:property name="base_ixx" value="8.2636e-04"/>
+  <xacro:property name="base_iyy" value="1.3056e-03"/>
+  <xacro:property name="base_izz" value="1.0732e-03"/>
+  <xacro:property name="base_ixy" value="3.7746e-06"/>
+  <xacro:property name="base_ixz" value="-4.2957e-05"/>
+  <xacro:property name="base_iyz" value="-1.5498e-06"/>
+  <xacro:property name="coxa_mass" value="0.0200143"/>
+  <xacro:property name="coxa_cx" value="-0.00178525"/>
+  <xacro:property name="coxa_cy" value="0.0295615"/>
+  <xacro:property name="coxa_cz" value="-0.00439371"/>
+  <xacro:property name="coxa_ixx" value="4.0522e-06"/>
+  <xacro:property name="coxa_iyy" value="3.0828e-06"/>
+  <xacro:property name="coxa_izz" value="3.3662e-06"/>
+  <xacro:property name="coxa_ixy" value="2.0280e-07"/>
+  <xacro:property name="coxa_ixz" value="1.3216e-08"/>
+  <xacro:property name="coxa_iyz" value="2.5010e-07"/>
+  <xacro:property name="femur_mass" value="0.00891947"/>
+  <xacro:property name="femur_cx" value="-0.00630845"/>
+  <xacro:property name="femur_cy" value="0.0278224"/>
+  <xacro:property name="femur_cz" value="5.95122e-10"/>
+  <xacro:property name="femur_ixx" value="2.7866e-06"/>
+  <xacro:property name="femur_iyy" value="2.8842e-06"/>
+  <xacro:property name="femur_izz" value="5.3800e-06"/>
+  <xacro:property name="femur_ixy" value="1.4510e-08"/>
+  <xacro:property name="femur_ixz" value="5.3652e-14"/>
   <xacro:property name="femur_iyz" value="-6.8104e-12"/>
-  <xacro:property name="tibia_mass" value="0.0185889"/>
-  <xacro:property name="tibia_cx" value="-0.00308253"/>
-  <xacro:property name="tibia_cy" value="0.000845768"/>
-  <xacro:property name="tibia_cz" value="-0.0100566"/>
-  <xacro:property name="tibia_ixx" value="6.3377e-06"/>
-  <xacro:property name="tibia_iyy" value="7.1075e-06"/>
-  <xacro:property name="tibia_izz" value="1.4382e-06"/>
-  <xacro:property name="tibia_ixy" value="-1.5538e-08"/>
-  <xacro:property name="tibia_ixz" value="-2.1874e-07"/>
-  <xacro:property name="tibia_iyz" value="1.2982e-07"/>
+  <xacro:property name="tibia_mass" value="0.0179021"/>
+  <xacro:property name="tibia_cx" value="-0.00325911"/>
+  <xacro:property name="tibia_cy" value="0.00066042"/>
+  <xacro:property name="tibia_cz" value="-0.00898153"/>
+  <xacro:property name="tibia_ixx" value="5.0764e-06"/>
+  <xacro:property name="tibia_iyy" value="5.8392e-06"/>
+  <xacro:property name="tibia_izz" value="1.3679e-06"/>
+  <xacro:property name="tibia_ixy" value="-1.3773e-08"/>
+  <xacro:property name="tibia_ixz" value="-1.3394e-07"/>
+  <xacro:property name="tibia_iyz" value="1.1033e-07"/>
 </robot>
